Commit message: Added collision models

File: sr_scara_hx_description/urdf/sr_scara_hx.urdf (robot description, URDF)
Before this commit: robot sr_scara_hx, 4 links, 3 joints
Links:
- link base_link: geometry collision mesh filename=package://sr_scara_hx_description/meshes/base.stl scale=0.001 0.001 0.001; visual mesh filename=package://sr_scara_hx_description/meshes/base.stl scale=0.001 0.001 0.001
- link link1: geometry collision mesh filename=package://sr_scara_hx_description/meshes/link1.stl scale=0.001 0.001 0.001; visual mesh filename=package://sr_scara_hx_description/meshes/link1.stl scale=0.001 0.001 0.001
- link link2: geometry collision mesh filename=package://sr_scara_hx_description/meshes/link2.stl scale=0.001 0.001 0.001; visual mesh filename=package://sr_scara_hx_description/meshes/link2.stl scale=0.001 0.001 0.001
- link probe: geometry collision mesh filename=package://sr_scara_hx_description/meshes/probe.stl scale=0.001 0.001 0.001; visual mesh filename=package://sr_scara_hx_description/meshes/probe.stl scale=0.001 0.001 0.001

Commit message: gripper_base added

File: sr_scara_hx_description/urdf/sr_scara_hx.urdf (robot description, URDF)
Before this commit: robot sr_scara_hx, 4 links, 3 joints
Links:
- added link gripper_base; visual box size=0.06 .02 .01
Joints:
- added joint gripper_con: type fixed, parent probe, child gripper_base, origin xyz=0 0 0 rpy=0 0 0

Commit message: urdf update-dummy gripper, moveit rviz plugin ok

File: sr_scara_hx_description/urdf/sr_scara_hx.urdf (robot description, URDF)
Before this commit: robot sr_scara_hx, 5 links, 4 joints
Links:
- added link gripper_dummy; visual box size=0.06 .02 .01
Joints:
- added joint gripper_dummy: type fixed, parent gripper_base, child gripper_dummy, origin xyz=0 0 0 rpy=0 0 0
- joint gripper_con: axis (none) -> 0 0 1; limit (none) -> lower=-3 upper=3 effort=3.0 velocity=0.01; type fixed -> revolute
